File: hardware/macropad_synthplug.sch (EAGLE design)
At the start: 13 parts, among them IC1 H11L1MS, J1 SJ-3523-SMT, J2 SJ-3523-SMT

Commit message: added sch pdf
Other:
- note added: "2022 @todbot / Tod Kurt"
Changed lines of the file:
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@@
 <part name="+3V2" library="supply1" library_urn="urn:adsk.eagle:library:371" deviceset="+3V3" device=""/>
 <part name="D1" library="diode" library_urn="urn:adsk.eagle:library:210" deviceset="DIODE-" device="SOD123" package3d_urn="urn:adsk.eagle:package:43420/1" value="1N4148"/>
+<part name="FRAME2" library="frames" library_urn="urn:adsk.eagle:library:229" deviceset="A4L-LOC" device="" value="test"/>
 </parts>
 <sheets>
@@
 - SCL - GP21 - UART1 RX - PWM2A</text>
 <text x="-10.16" y="22.86" size="1.778" layer="97">From Figure 3.4.1 of "Hardware Design with RP2040" </text>
+<text x="71.12" y="-22.86" size="2.1844" layer="94" ratio="13">2022 @todbot / Tod Kurt</text>
 </plain>
 <instances>
@@
 <attribute name="VALUE" x="34.0614" y="74.676" size="1.778" layer="96" rot="R90"/>
 </instance>
+<instance part="FRAME2" gate="G$1" x="-93.98" y="-27.94" smashed="yes">
+<attribute name="DRAWING_NAME" x="123.19" y="-12.7" size="2.54" layer="94"/>
+<attribute name="LAST_DATE_TIME" x="123.19" y="-17.78" size="2.286" layer="94"/>
+<attribute name="SHEET" x="136.525" y="-22.86" size="2.54" layer="94"/>
+</instance>
 </instances>
